File: wledcar.kicad_sch (KiCad schematic)
At the start: 35 parts, among them J1 Conn_01x04, J2 USB_C_Receptacle_USB2.0_16P, J3 Screw_Terminal_01x02, J4 Screw_Terminal_01x02, SW1 SW_SPDT, U1 SN74AHCT125N, U2 XL4015, U3 AMS1117-3.3, U4 ESP32-S3-WROOM-1

Commit message: Add files via upload
Parts:
- removed J4: Screw_Terminal_01x02, symbol Connector:Screw_Terminal_01x02
- removed SW1: SW_SPDT, symbol Switch:SW_SPDT
- added C12: 1uF, Capacitor_SMD:C_0603_1608Metric, symbol Device:C_Small
- added D1, D3: SS54, PCM_JLCPCB:D_SMA, symbol PCM_JLCPCB-Diodes:Schottky,SS54
- added J8: Screw_Terminal_01x08, TerminalBlock_Phoenix:TerminalBlock_Phoenix_MKDS-3-8-5.08_1x08_P5.08mm_Horizontal, symbol Connector:Screw_Terminal_01x08
- C1, C10, C2, C3, C4, C5, C6, C7, C8, C9: footprint (none) -> Capacitor_SMD:C_0603_1608Metric
- C11: value 0.1uF -> 1uF; footprint (none) -> Capacitor_SMD:C_0603_1608Metric
- J1: footprint (none) -> Connector_PinHeader_1.27mm:PinHeader_1x04_P1.27mm_Vertical
- J2: footprint (none) -> Connector_USB:USB_C_Receptacle_HRO_TYPE-C-31-M-12
- J3: footprint (none) -> TerminalBlock_Phoenix:TerminalBlock_Phoenix_MKDS-1,5-2-5.08_1x02_P5.08mm_Horizontal
- JP1, JP2: footprint (none) -> Jumper:SolderJumper-2_P1.3mm_Open_RoundedPad1.0x1.5mm
- L1: footprint Inductor_SMD:L_Vishay_IHLP-6767 -> Inductor_SMD:L_APV_APH1265
- R1, R2, R3, R4, R5, R6, R7, R8, R9: footprint (none) -> Resistor_SMD:R_0603_1608Metric
- R10: value 3.3k -> 1k; footprint (none) -> Resistor_SMD:R_0603_1608Metric
- R11: value 10k -> 3.3k; footprint (none) -> Resistor_SMD:R_0603_1608Metric
- U1: footprint N14 -> Package_SO:SOIC-14_3.9x8.7mm_P1.27mm
Connections:
- net +12V: now also C11.2
- net GND: now also C12.1
- net LED1: now also J8.2 (Pin_2)
- net LED2: now also J8.4 (Pin_4)
- net LED3: now also J8.6 (Pin_6)
- net LED4: now also J8.8 (Pin_8)
- net LED5V: now also C1.1, C2.1, U3.3 (VI), U4.2 (3V3), D1.1, D3.1, J8.1 (Pin_1), J8.3 (Pin_3), J8.5 (Pin_5), J8.7 (Pin_7)
- net MCULED1: now also U4.19 (IO11); no longer U4.39 (IO1)
- net MCULED2: now also U4.20 (IO12); no longer U4.38 (IO2)
- net MCULED3: now also U4.21 (IO13); no longer U4.15 (IO3)
- net MCULED4: now also U4.22 (IO14); no longer U4.4 (IO4)
- net VBUS: now also D3.2; no longer C1.1, C2.1, U3.3 (VI)
- net VDD: no longer U4.2 (3V3)
- net c5V: now also C12.2, D1.2; no longer C11.2, R10.2
- net at R11.1, U2.2 (FB): now also R10.2
Other:
- moved on the sheet: C8, C9, D2, L1, R10, R11

Commit message: update
Parts:
- removed C5, C6: 0.1uF, Capacitor_SMD:C_0603_1608Metric, symbol Device:C_Small
Changed lines of the file:
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@@
 	(paper "A4")
 	(junction
-		(at 33.02 69.85)
-		(diameter 0)
-		(color 0 0 0 0)
-	)
-	(junction
-		(at 33.02 77.47)
-		(diameter 0)
-		(color 0 0 0 0)
-	)
-	(junction
 		(at 151.13 125.73)
 		(diameter 0)
@@
 	)
 	(junction
-		(at 45.72 81.28)
-		(diameter 0)
-		(color 0 0 0 0)
-	)
-	(junction
 		(at 147.32 63.5)
 		(diameter 0)
@@
 	)
 	(junction
-		(at 45.72 73.66)
-		(diameter 0)
-		(color 0 0 0 0)
-	)
-	(junction
 		(at 186.69 63.5)
 		(diameter 0)
@@
 	(wire
 		(pts
-			(xy 29.21 69.85) (xy 33.02 69.85)
-		)
-		(stroke
-			(width 0)
-			(type default)
-		)
-	)
-	(wire
-		(pts
 			(xy 52.07 156.21) (xy 52.07 158.75)
 		)
@@
 	(wire
 		(pts
-			(xy 41.91 81.28) (xy 45.72 81.28)
-		)
-		(stroke
-			(width 0)
-			(type default)
-		)
-	)
-	(wire
-		(pts
 			(xy 92.71 99.06) (xy 96.52 99.06)
 		)
@@
 	(wire
 		(pts
-			(xy 41.91 73.66) (xy 45.72 73.66)
-		)
-		(stroke
-			(width 0)
-			(type default)
-		)
-	)
-	(wire
-		(pts
 			(xy 24.13 22.86) (xy 30.48 22.86)
 		)
@@
 	(wire
 		(pts
-			(xy 29.21 77.47) (xy 33.02 77.47)
-		)
-		(stroke
-			(width 0)
-			(type default)
-		)
-	)
-	(wire
-		(pts
 			(xy 76.2 36.83) (xy 76.2 27.94)
 		)
@@
 	(wire
 		(pts
-			(xy 29.21 71.12) (xy 29.21 69.85)
-		)
-		(stroke
-			(width 0)
-			(type default)
-		)
-	)
-	(wire
-		(pts
 			(xy 185.42 63.5) (xy 186.69 63.5)
 		)
@@
 	(wire
 		(pts
-			(xy 41.91 74.93) (xy 41.91 73.66)
-		)
-		(stroke
-			(width 0)
-			(type default)
-		)
-	)
-	(wire
-		(pts
 			(xy 92.71 96.52) (xy 96.52 96.52)
 		)
@@
 	(wire
 		(pts
-			(xy 29.21 76.2) (xy 29.21 77.47)
-		)
-		(stroke
-			(width 0)
-			(type default)
-		)
-	)
-	(wire
-		(pts
 			(xy 33.02 68.58) (xy 62.23 68.58)
 		)
@@
 	(wire
 		(pts
-			(xy 41.91 80.01) (xy 41.91 81.28)
-		)
-		(stroke
-			(width 0)
-			(type default)
-		)
-	)
-	(wire
-		(pts
 			(xy 67.31 22.86) (xy 76.2 22.86)
 		)
@@
 	(symbol
 		(lib_id "Device:C_Small")
-		(at 29.21 73.66 180)
-		(unit 1)
-		(exclude_from_sim no)
-		(in_bom yes)
-		(on_board yes)
-		(dnp no)
-		(property "Reference" "C5"
-			(at 23.368 73.152 0)
-			(effects
-				(font
-					(size 1.27 1.27)
-				)
-				(justify right)
-			)
-		)
-		(property "Value" "0.1uF"
-			(at 23.368 75.692 0)
-			(effects
-				(font
-					(size 1.27 1.27)
-				)
-				(justify right)
-			)
-		)
-		(property "Footprint" "Capacitor_SMD:C_0603_1608Metric"
-			(at 29.21 73.66 0)
-			(effects
-				(font
-					(size 1.27 1.27)
-				)
-				(hide yes)
-			)
-		)
-		(property "Datasheet" "~"
-			(at 29.21 73.66 0)
-			(effects
-				(font
-					(size 1.27 1.27)
-				)
-				(hide yes)
-			)
-		)
-		(property "Description" "Unpolarized capacitor, small symbol"
-			(at 29.21 73.66 0)
-			(effects
-				(font
-					(size 1.27 1.27)
-				)
-				(hide yes)
-			)
-		)
-		(pin "1"
-		)
-		(pin "2"
-		)
-		(instances
-			(project ""
-				(path "/7d92a72b-2c0c-4602-8f3f-8951598714e4"
-					(reference "C5")
-					(unit 1)
-				)
-			)
-		)
-	)
-	(symbol
-		(lib_id "Device:C_Small")
 		(at 147.32 72.39 180)
 		(unit 1)
@@
 					(unit 1)
 				)
-			)
-		)
-	)
-	(symbol
-		(lib_id "Device:C_Small")
-		(at 41.91 77.47 180)
-		(unit 1)
-		(exclude_from_sim no)
-		(in_bom yes)
-		(on_board yes)
-		(dnp no)
-		(property "Reference" "C6"
-			(at 36.576 76.962 0)
-			(effects
-				(font
-					(size 1.27 1.27)
-				)
-				(justify right)
-			)
-		)
-		(property "Value" "0.1uF"
-			(at 36.576 79.502 0)
-			(effects
-				(font
-					(size 1.27 1.27)
-				)
-				(justify right)
-			)
-		)
-		(property "Footprint" "Capacitor_SMD:C_0603_1608Metric"
-			(at 41.91 77.47 0)
-			(effects
-				(font
-					(size 1.27 1.27)
-				)
-				(hide yes)
-			)
-		)
-		(property "Datasheet" "~"
-			(at 41.91 77.47 0)
-			(effects
-				(font
-					(size 1.27 1.27)
-				)
-				(hide yes)
-			)
-		)
-		(property "Description" "Unpolarized capacitor, small symbol"
-			(at 41.91 77.47 0)
-			(effects
-				(font
-					(size 1.27 1.27)
-				)
-				(hide yes)
-			)
-		)
-		(pin "1"
-		)
-		(pin "2"
-		)
-		(instances
-			(project "wledcar"
-				(path "/7d92a72b-2c0c-4602-8f3f-8951598714e4"
-					(reference "C6")
-					(unit 1)
-				)

Commit message: redid the whole pcb 	modified:   wledcar.kicad_pcb 	modified:   wledcar.kicad_pro 	modified:   wledcar.kicad_sch
Connections:
- net +12V: now also J3.2 (Pin_2); no longer J3.1 (Pin_1)
- net GND: now also J3.1 (Pin_1); no longer J3.2 (Pin_2)
Changed lines of the file:
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@@
 	(global_label "+12V"
 		(shape input)
-		(at 156.21 97.79 180)
+		(at 156.21 100.33 180)
 		(fields_autoplaced yes)
 		(effects
@@
 		)
 		(property "Intersheetrefs" "${INTERSHEET_REFS}"
-			(at 148.1448 97.79 0)
+			(at 148.1448 100.33 0)
 			(effects
 				(font
@@
 	(symbol
 		(lib_id "power:GND")
-		(at 156.21 100.33 270)
+		(at 156.21 97.79 270)
 		(unit 1)
 		(exclude_from_sim no)
@@
 		(dnp no)
 		(property "Reference" "#PWR016"
-			(at 149.86 100.33 0)
+			(at 149.86 97.79 0)
 			(effects
 				(font
@@
 		)
 		(property "Value" "GND"
-			(at 152.4 100.3301 90)
+			(at 152.4 97.7901 90)
 			(effects
 				(font
@@
 		)
 		(property "Footprint" ""
-			(at 156.21 100.33 0)
+			(at 156.21 97.79 0)
 			(effects
 				(font
@@
 		)
 		(property "Datasheet" ""
-			(at 156.21 100.33 0)
+			(at 156.21 97.79 0)
 			(effects
 				(font
@@
 		)
 		(property "Description" "Power symbol creates a global label with name \"GND\" , ground"
-			(at 156.21 100.33 0)
+			(at 156.21 97.79 0)
 			(effects
 				(font

Commit message: did some cyaoing 	modified:   wledcar.kicad_pcb 	modified:   wledcar.kicad_pro 	modified:   wledcar.kicad_sch
Connections:
- net USB_D+: now reaches R5.1, U4.14 (USB_D+)
- net USB_D-: now reaches R4.1, U4.13 (USB_D-)
Other:
- moved on the sheet: R4, R5
Changed lines of the file:
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@@
 	(wire
 		(pts
-			(xy 97.79 81.28) (xy 111.76 81.28)
+			(xy 104.14 81.28) (xy 111.76 81.28)
 		)
 		(stroke
@@
 	(wire
 		(pts
+			(xy 99.06 78.74) (xy 92.71 78.74)
+		)
+		(stroke
+			(width 0)
+			(type default)
+		)
+	)
+	(wire
+		(pts
 			(xy 67.31 36.83) (xy 67.31 27.94)
 		)
@@
 	(wire
 		(pts
+			(xy 99.06 81.28) (xy 92.71 81.28)
+		)
+		(stroke
+			(width 0)
+			(type default)
+		)
+	)
+	(wire
+		(pts
 			(xy 195.58 78.74) (xy 205.74 78.74)
 		)
@@
 	(wire
 		(pts
-			(xy 97.79 78.74) (xy 111.76 78.74)
+			(xy 104.14 78.74) (xy 111.76 78.74)
 		)
 		(stroke
@@
 		)
 	)
+	(global_label "USB_D+"
+		(shape input)
+		(at 96.52 81.28 270)
+		(fields_autoplaced yes)
+		(effects
+			(font
+				(size 1.27 1.27)
+			)
+			(justify right)
+		)
+		(property "Intersheetrefs" "${INTERSHEET_REFS}"
+			(at 96.52 91.8852 90)
+			(effects
+				(font
+					(size 1.27 1.27)
+				)
+				(justify right)
+				(hide yes)
+			)
+		)
+	)
 	(global_label "D+"
 		(shape input)
@@
 		(property "Intersheetrefs" "${INTERSHEET_REFS}"
 			(at 117.5876 78.74 0)
+			(effects
+				(font
+					(size 1.27 1.27)
+				)
+				(justify left)
+				(hide yes)
+			)
+		)
+	)
+	(global_label "USB_D-"
+		(shape input)
+		(at 96.52 78.74 90)
+		(fields_autoplaced yes)
+		(effects
+			(font
+				(size 1.27 1.27)
+			)
+			(justify left)
+		)
+		(property "Intersheetrefs" "${INTERSHEET_REFS}"
+			(at 96.52 68.1348 90)
 			(effects
 				(font
@@
 	(symbol
 		(lib_id "Device:R_Small")
-		(at 95.25 81.28 90)
+		(at 101.6 81.28 90)
 		(unit 1)
 		(exclude_from_sim no)
@@
 		(dnp no)
 		(property "Reference" "R5"
-			(at 98.298 83.312 90)
+			(at 104.648 83.312 90)
 			(effects
 				(font
@@
 		)
 		(property "Value" "22"
-			(at 98.298 85.852 90)
+			(at 104.648 85.852 90)
 			(effects
 				(font
@@
 		)
 		(property "Footprint" "Resistor_SMD:R_0603_1608Metric"
-			(at 95.25 81.28 0)
+			(at 101.6 81.28 0)
 			(effects
 				(font
@@
 		)
 		(property "Datasheet" "~"
-			(at 95.25 81.28 0)
+			(at 101.6 81.28 0)
 			(effects
 				(font
@@
 		)
 		(property "Description" "Resistor, small symbol"
-			(at 95.25 81.28 0)
+			(at 101.6 81.28 0)
 			(effects
 				(font
@@
 	(symbol
 		(lib_id "Device:R_Small")
-		(at 95.25 78.74 90)
+		(at 101.6 78.74 90)
 		(unit 1)
 		(exclude_from_sim no)
@@
 		(dnp no)
 		(property "Reference" "R4"
-			(at 97.536 73.66 90)
+			(at 103.886 73.66 90)
 			(effects
 				(font
@@
 		)
 		(property "Value" "22"
-			(at 97.536 76.2 90)
+			(at 103.886 76.2 90)
 			(effects
 				(font
@@
 		)
 		(property "Footprint" "Resistor_SMD:R_0603_1608Metric"
-			(at 95.25 78.74 0)
+			(at 101.6 78.74 0)
 			(effects
 				(font
@@
 		)
 		(property "Datasheet" "~"
-			(at 95.25 78.74 0)
+			(at 101.6 78.74 0)
 			(effects
 				(font
@@
 		)
 		(property "Description" "Resistor, small symbol"
-			(at 95.25 78.74 0)
-			(effects
-				(font
+			(at 101.6 78.74 0)
+			(effects
+				(font

Commit message: moar update 	modified:   wledcar.kicad_pcb 	modified:   wledcar.kicad_pro 	modified:   wledcar.kicad_sch
Connections:
- net SW: now reaches D2.1, L1.1, U2.3 (SW)
Changed lines of the file:
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@@
+		)
+	)
+	(global_label "SW"
+		(shape input)
+		(at 177.8 63.5 90)
+		(fields_autoplaced yes)
+		(effects
+			(font
+				(size 1.27 1.27)
+			)
+			(justify left)
+		)
+		(property "Intersheetrefs" "${INTERSHEET_REFS}"
+			(at 177.8 57.8539 90)
+			(effects
+				(font
+					(size 1.27 1.27)
+				)
+				(justify left)
+				(hide yes)
+			)
 		)
 	)
