File: wledcar.kicad_pcb (KiCad board)
At the start: 2 copper layers, 41.6 x 46.2 mm, 37 parts, among them J1 Conn_01x04, J2 USB_C_Receptacle_USB2.0_16P, J3 Screw_Terminal_01x02, J8 Screw_Terminal_01x08, U1 SN74AHCT125N, U2 XL4015, U3 AMS1117-3.3, U4 ESP32-S3-WROOM-1

Commit message: update
Parts:
- removed C5, C6: 0.1uF, Capacitor_SMD:C_0603_1608Metric
- moved C8 9.06 mm to (211.3, 129.8), turned to 90 degrees
- moved C11 6.65 mm to (212.8, 129.8), turned to 90 degrees
- moved D2 4.69 mm to (218.6, 125.3)
- moved C9 2.26 mm to (229.2, 122.4), turned to 90 degrees
- moved L1 2.12 mm to (223.3, 114.2)
- moved R10 0.08 mm to (212.9, 116.0), turned to 180 degrees
- moved R11 0.08 mm to (212.9, 114.4), turned to 0 degrees
- turned C12 to 90 degrees
Routing:
- net +12V: track 30.3 -> 44.4 mm, vias 1 -> 2
- net GND: track 18.0 -> 12.1 mm, vias 15 -> 23
- net c5V: track 38.8 -> 44.2 mm
- net Net-(JP1-B): track 12.4 -> 9.36 mm
- net Net-(JP2-B): track 5.81 -> 3.76 mm
- net Net-(U2-FB): track 12.3 -> 10.7 mm
- net LED1: track 26.7 -> 25.5 mm
- net MCULED2: track 10.8 -> 11.4 mm

Commit message: redid the whole pcb 	modified:   wledcar.kicad_pcb 	modified:   wledcar.kicad_pro 	modified:   wledcar.kicad_sch
Parts:
- J1: moved to B.Cu
- JP2: moved to F.Cu
- moved C1 26.9 mm to (211.6, 92.7), turned to 90 degrees
- moved C2 26.0 mm to (210.0, 92.7), turned to 90 degrees
- moved C3 22.9 mm to (214.7, 92.7)
- moved C4 22.9 mm to (213.1, 92.7)
- moved J1 19.3 mm to (238.6, 101.7)
- moved U3 18.4 mm to (213.5, 104.5), turned to -90 degrees
- moved D3 17.7 mm to (204.4, 117.2), turned to 90 degrees
- moved D1 14.6 mm to (200.9, 117.2), turned to 90 degrees
- moved C8 11.9 mm to (223.2, 129.5), turned to 180 degrees
- moved R10 11.3 mm to (221.8, 122.9)
- moved R11 11.3 mm to (221.8, 121.3)
- moved C9 11.2 mm to (224.3, 112.3), turned to 180 degrees
- moved C11 10.6 mm to (223.2, 128.0), turned to 180 degrees
- moved R6 9.35 mm to (229.7, 116.9), turned to 90 degrees
- moved C12 9.12 mm to (224.3, 113.9), turned to 180 degrees
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Connections:
- J3 pad 1: +12V -> GND
- J3 pad 2: GND -> +12V
Routing:
- net LED1: track 25.5 -> 52.7 mm
- net LED2: track 11.2 -> 38.0 mm
- net VDD: track 44.5 -> 18.0 mm
- net Net-(J1-Pin_4): track 26.2 -> 1.95 mm
- net Net-(J1-Pin_3): track 23.2 -> 1.95 mm
- net Net-(J1-Pin_2): track 20.3 -> 1.95 mm
- net Net-(J1-Pin_1): track 16.8 -> 1.95 mm
- net LED3: track 11.9 -> 20.8 mm
- net +12V: track 44.4 -> 52.8 mm, vias 2 -> 0
- net GND: track 12.1 -> 4.62 mm, vias 23 -> 124
- net Net-(U2-FB): track 10.7 -> 5.13 mm
- net MCULED1: track 7.46 -> 12.9 mm
- net MCULED2: track 11.4 -> 16.6 mm
- net MCULED3: track 12.4 -> 17.4 mm
- net Net-(JP1-B): track 9.36 -> 4.47 mm, vias 2 -> 0
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Other:
- board size 41.6 x 46.2 mm -> 41.7 x 50 mm

Commit message: did some cyaoing 	modified:   wledcar.kicad_pcb 	modified:   wledcar.kicad_pro 	modified:   wledcar.kicad_sch
Parts:
- moved D1 3.50 mm to (204.4, 117.2)
- moved D3 3.50 mm to (200.9, 117.2)
- moved C3 3.10 mm to (214.8, 95.8)
- moved C1 3.10 mm to (211.7, 95.8)
- moved C2 3.10 mm to (210.1, 95.8)
- moved C4 3.10 mm to (213.2, 95.8)
- moved U3 2.83 mm to (213.9, 101.7)
Connections:
- net Net-(U4-USB_D+) renamed USB_D+
- net Net-(U4-USB_D-) renamed USB_D-
Routing:
- net LED1: track 52.7 -> 29.8 mm
- net LED2: track 38.0 -> 18.1 mm
- net c5V: track 48.0 -> 41.5 mm
- net LED5V: track 119.0 -> 113.4 mm
- net LED3: track 20.8 -> 17.1 mm
- net VBUS: track 27.1 -> 26.1 mm
- net VDD: track 18.0 -> 17.2 mm, vias 2 -> 0
- net USB_D-: track 15.9 -> 16.7 mm
- net GND: vias 124 -> 178

Commit message: moar update 	modified:   wledcar.kicad_pcb 	modified:   wledcar.kicad_pro 	modified:   wledcar.kicad_sch
Connections:
- net Net-(U2-SW) renamed SW
Routing:
- net SW: track 29.9 -> 2.12 mm
- net LED5V: track 113.4 -> 106.2 mm
- net GND: vias 178 -> 40
- added copper zone on B.Cu, net SW

Commit message: few edits 	modified:   wledcar.kicad_pcb
Routing:
- net LED1: track 29.8 -> 35.2 mm
- net LED2: track 18.1 -> 22.1 mm
- net GND: vias 40 -> 314
